Commit message: made some package names actually match folder names

File: simulation/swapbot.urdf.xacro (robot description, xacro)
@@ -22,5 +22,5 @@
     <visual>
       <geometry>
-	<mesh filename= "package://robot_simulation/betterbase.stl" scale="0.0254 0.0254 0.0254"/>
+	<mesh filename= "package://simulation/betterbase.stl" scale="0.0254 0.0254 0.0254"/>
         <!--<box size="${blength} ${bwidth} ${bheight}"/>-->
       </geometry>
@@ -32,5 +32,5 @@
     <collision>
       <geometry>
-	<mesh filename= "package://robot_simulation/betterbase.stl" scale="0.0254 0.0254 0.0254"/>
+	<mesh filename= "package://simulation/betterbase.stl" scale="0.0254 0.0254 0.0254"/>
         <!--<box size="${blength} ${bwidth} ${bheight}"/>-->
       </geometry>

Commit message: Fixed simulated drive

File: simulation/swapbot.urdf.xacro (robot description, xacro)
@@ -10,13 +10,7 @@
     <inertial>
       <mass value="${mass}" />
-      <inertia ixx="0.1" ixy="0.0" ixz="0.0" iyy="0.1" iyz="0.0" izz="0.1" />
+      <inertia ixx="0.01" ixy="0.0" ixz="0.0" iyy="0.01" iyz="0.0" izz="0.01" />
     </inertial>
   </xacro:macro>
-  <!-- MoveIt requires a fixed base for the arm -->
-  <link name="dummy_base"/>
-  <joint name="dummy_joint" type="fixed">
-     <parent link="dummy_base"/>
-     <child link="base_link"/>
-  </joint>
   <link name="base_link">
     <visual>
@@ -42,83 +36,4 @@
     <xacro:default_inertial mass="50"/>
   </link>
-  <xacro:macro name="m_joint" params="name type axis_xyz origin_rpy origin_xyz parent child limit_e limit_l limit_u limit_v">
-    <joint name="${name}" type="${type}">
-      <axis xyz="${axis_xyz}" />
-      <limit effort="${limit_e}" lower="${limit_l}" upper="${limit_u}" velocity="${limit_v}" />
-      <origin rpy="${origin_rpy}" xyz="${origin_xyz}" />
-      <parent link="${parent}" />
-      <child link="${child}" />
-    </joint>
-    <transmission name="trans_${name}">
-      <type>transmission_interface/SimpleTransmission</type>
-      <joint name="${name}">
-        <hardwareInterface>hardware_interface/PositionJointInterface</hardwareInterface>
-      </joint>
-      <actuator name="motor_${name}">
-        <hardwareInterface>hardware_interface/PositionJointInterface</hardwareInterface>
-        <mechanicalReduction>1</mechanicalReduction>
-      </actuator>
-    </transmission>
-  </xacro:macro>
-  <xacro:macro name="m_link_cylinder" params="name origin_xyz origin_rpy radius length mass ixx ixy ixz iyy iyz izz">
-    <link name="${name}">
-      <inertial>
-        <mass value="${mass}" />
-        <origin rpy="${origin_rpy}" xyz="${origin_xyz}" />
-        <inertia ixx="${ixx}" ixy="${ixy}" ixz="${ixz}" iyy="${iyy}" iyz="${iyz}" izz="${izz}" />
-      </inertial>
-      <collision>
-        <origin rpy="${origin_rpy}" xyz="${origin_xyz}*0.9" />
-        <geometry>
-          <cylinder radius="${radius}*0.9" length="${length}*0.9" />
-        </geometry>
-      </collision>
-      <visual>
-        <origin rpy="${origin_rpy}" xyz="${origin_xyz}" />
-        <geometry>
-          <cylinder radius="${radius}" length="${length}" />
-        </geometry>
-        <material name="blue">
-          <color rgba="0 0 1 1"/>
-        </material>
-      </visual>
-    </link>
-  </xacro:macro>
-  <m_joint name="base_to_arm_1" type="revolute"
-           axis_xyz="0 1 0"
-           origin_rpy="0 0 0" origin_xyz="-0.4 0 0.15"
-           parent="base_link" child="arm_1"
-           limit_e="1000" limit_l="-3.14" limit_u="3.14" limit_v="0.5" />
-  <m_link_cylinder name="arm_1"
-              origin_rpy="0 0 0" origin_xyz="0 0 0.206"
-              mass="1"
-              ixx="0.01" ixy="0" ixz="0"
-              iyy="0.01" iyz="0"
-              izz="0.01"
-              radius="0.02" length="0.413" />
-  <m_joint name="arm_1_to_arm_2" type="revolute"
-           axis_xyz="0 1 0"
-           origin_rpy="0 0 0" origin_xyz="0 0 0.413"
-           parent="arm_1" child="arm_2"
-           limit_e="1000" limit_l="-3.14" limit_u="3.14" limit_v="0.5" />
-  <m_link_cylinder name="arm_2"
-              origin_rpy="0 0 0" origin_xyz="0 0 0.182"
-              mass="1"
-              ixx="0.01" ixy="0" ixz="0"
-              iyy="0.01" iyz="0"
-              izz="0.01"
-              radius="0.02" length="0.365" />
-  <m_joint name="arm_2_to_arm_3" type="revolute"
-           axis_xyz="0 1 0"
-           origin_rpy="0 0 0" origin_xyz="0 0 0.365"
-           parent="arm_2" child="arm_3"
-           limit_e="1000" limit_l="-3.14" limit_u="3.14" limit_v="0.5" />
-  <m_link_cylinder name="arm_3"
-              origin_rpy="0 0 0" origin_xyz="0 0 0.05"
-              mass="1"
-              ixx="0.01" ixy="0" ixz="0"
-              iyy="0.01" iyz="0"
-              izz="0.01"
-              radius="0.02" length="0.1" />
   <xacro:macro name="wheel" params="prefix suffix ref ref2">
     <link name="${prefix}_${suffix}_wheel">
@@ -153,5 +68,5 @@
     <gazebo reference="${prefix}_${suffix}_wheel">
       <fdir1 value="0 0 1"/>
-      <mu1 value="1"/>
+      <mu1 value="0.1"/>
       <mu2 value="100"/>
       <kp value="10000000.0" />

Commit message: Revert "Fixed simulated drive"
This reverts commit 064bef770697d85c45fa1c162b8fa75f142f9008.

File: simulation/swapbot.urdf.xacro (robot description, xacro)
@@ -10,7 +10,13 @@
     <inertial>
       <mass value="${mass}" />
-      <inertia ixx="0.01" ixy="0.0" ixz="0.0" iyy="0.01" iyz="0.0" izz="0.01" />
+      <inertia ixx="0.1" ixy="0.0" ixz="0.0" iyy="0.1" iyz="0.0" izz="0.1" />
     </inertial>
   </xacro:macro>
+  <!-- MoveIt requires a fixed base for the arm -->
+  <link name="dummy_base"/>
+  <joint name="dummy_joint" type="fixed">
+     <parent link="dummy_base"/>
+     <child link="base_link"/>
+  </joint>
   <link name="base_link">
     <visual>
@@ -36,4 +42,83 @@
     <xacro:default_inertial mass="50"/>
   </link>
+  <xacro:macro name="m_joint" params="name type axis_xyz origin_rpy origin_xyz parent child limit_e limit_l limit_u limit_v">
+    <joint name="${name}" type="${type}">
+      <axis xyz="${axis_xyz}" />
+      <limit effort="${limit_e}" lower="${limit_l}" upper="${limit_u}" velocity="${limit_v}" />
+      <origin rpy="${origin_rpy}" xyz="${origin_xyz}" />
+      <parent link="${parent}" />
+      <child link="${child}" />
+    </joint>
+    <transmission name="trans_${name}">
+      <type>transmission_interface/SimpleTransmission</type>
+      <joint name="${name}">
+        <hardwareInterface>hardware_interface/PositionJointInterface</hardwareInterface>
+      </joint>
+      <actuator name="motor_${name}">
+        <hardwareInterface>hardware_interface/PositionJointInterface</hardwareInterface>
+        <mechanicalReduction>1</mechanicalReduction>
+      </actuator>
+    </transmission>
+  </xacro:macro>
+  <xacro:macro name="m_link_cylinder" params="name origin_xyz origin_rpy radius length mass ixx ixy ixz iyy iyz izz">
+    <link name="${name}">
+      <inertial>
+        <mass value="${mass}" />
+        <origin rpy="${origin_rpy}" xyz="${origin_xyz}" />
+        <inertia ixx="${ixx}" ixy="${ixy}" ixz="${ixz}" iyy="${iyy}" iyz="${iyz}" izz="${izz}" />
+      </inertial>
+      <collision>
+        <origin rpy="${origin_rpy}" xyz="${origin_xyz}*0.9" />
+        <geometry>
+          <cylinder radius="${radius}*0.9" length="${length}*0.9" />
+        </geometry>
+      </collision>
+      <visual>
+        <origin rpy="${origin_rpy}" xyz="${origin_xyz}" />
+        <geometry>
+          <cylinder radius="${radius}" length="${length}" />
+        </geometry>
+        <material name="blue">
+          <color rgba="0 0 1 1"/>
+        </material>
+      </visual>
+    </link>
+  </xacro:macro>
+  <m_joint name="base_to_arm_1" type="revolute"
+           axis_xyz="0 1 0"
+           origin_rpy="0 0 0" origin_xyz="-0.4 0 0.15"
+           parent="base_link" child="arm_1"
+           limit_e="1000" limit_l="-3.14" limit_u="3.14" limit_v="0.5" />
+  <m_link_cylinder name="arm_1"
+              origin_rpy="0 0 0" origin_xyz="0 0 0.206"
+              mass="1"
+              ixx="0.01" ixy="0" ixz="0"
+              iyy="0.01" iyz="0"
+              izz="0.01"
+              radius="0.02" length="0.413" />
+  <m_joint name="arm_1_to_arm_2" type="revolute"
+           axis_xyz="0 1 0"
+           origin_rpy="0 0 0" origin_xyz="0 0 0.413"
+           parent="arm_1" child="arm_2"
+           limit_e="1000" limit_l="-3.14" limit_u="3.14" limit_v="0.5" />
+  <m_link_cylinder name="arm_2"
+              origin_rpy="0 0 0" origin_xyz="0 0 0.182"
+              mass="1"
+              ixx="0.01" ixy="0" ixz="0"
+              iyy="0.01" iyz="0"
+              izz="0.01"
+              radius="0.02" length="0.365" />
+  <m_joint name="arm_2_to_arm_3" type="revolute"
+           axis_xyz="0 1 0"
+           origin_rpy="0 0 0" origin_xyz="0 0 0.365"
+           parent="arm_2" child="arm_3"
+           limit_e="1000" limit_l="-3.14" limit_u="3.14" limit_v="0.5" />
+  <m_link_cylinder name="arm_3"
+              origin_rpy="0 0 0" origin_xyz="0 0 0.05"
+              mass="1"
+              ixx="0.01" ixy="0" ixz="0"
+              iyy="0.01" iyz="0"
+              izz="0.01"
+              radius="0.02" length="0.1" />
   <xacro:macro name="wheel" params="prefix suffix ref ref2">
     <link name="${prefix}_${suffix}_wheel">
@@ -68,5 +153,5 @@
     <gazebo reference="${prefix}_${suffix}_wheel">
       <fdir1 value="0 0 1"/>
-      <mu1 value="0.1"/>
+      <mu1 value="1"/>
       <mu2 value="100"/>
       <kp value="10000000.0" />

Commit message: Fixed Xarco and rviz excavation launch

File: simulation/swapbot.urdf.xacro (robot description, xacro)
@@ -69,7 +69,7 @@
       </inertial>
       <collision>
-        <origin rpy="${origin_rpy}" xyz="${origin_xyz}*0.9" />
+        <origin rpy="${origin_rpy}" xyz="${origin_xyz}" />
         <geometry>
-          <cylinder radius="${radius}*0.9" length="${length}*0.9" />
+          <cylinder radius="${radius*0.9}" length="${length*0.9}" />
         </geometry>
       </collision>

Commit message: attempt at using a realsense in gazebo

File: simulation/swapbot.urdf.xacro (robot description, xacro)
@@ -13,10 +13,4 @@
     </inertial>
   </xacro:macro>
-  <!-- MoveIt requires a fixed base for the arm -->
-  <link name="dummy_base"/>
-  <joint name="dummy_joint" type="fixed">
-     <parent link="dummy_base"/>
-     <child link="base_link"/>
-  </joint>
   <link name="base_link">
     <visual>
@@ -42,4 +36,10 @@
     <xacro:default_inertial mass="50"/>
   </link>
+    <!-- Import macro for realsense-RS200 camera-->
+    <xacro:include filename="$(find realsense_gazebo_plugin)/urdf/realsense-RS200.macro.xacro"/>
+    <!-- Create camera instance -->
+    <xacro:realsense-rs200 prefix="" parent="base_link">
+        <origin xyz="0.45 0 0.15" rpy="0 0 0" />
+    </xacro:realsense-rs200>
   <xacro:macro name="m_joint" params="name type axis_xyz origin_rpy origin_xyz parent child limit_e limit_l limit_u limit_v">
     <joint name="${name}" type="${type}">

Commit message: updated some doc, also fixed an issue caused by some dick over at ros_control

File: simulation/swapbot.urdf.xacro (robot description, xacro)
@@ -36,10 +36,4 @@
     <xacro:default_inertial mass="50"/>
   </link>
-    <!-- Import macro for realsense-RS200 camera-->
-    <xacro:include filename="$(find realsense_gazebo_plugin)/urdf/realsense-RS200.macro.xacro"/>
-    <!-- Create camera instance -->
-    <xacro:realsense-rs200 prefix="" parent="base_link">
-        <origin xyz="0.45 0 0.15" rpy="0 0 0" />
-    </xacro:realsense-rs200>
   <xacro:macro name="m_joint" params="name type axis_xyz origin_rpy origin_xyz parent child limit_e limit_l limit_u limit_v">
     <joint name="${name}" type="${type}">

Commit message: working realsense_camera

File: simulation/swapbot.urdf.xacro (robot description, xacro)
@@ -36,4 +36,10 @@
     <xacro:default_inertial mass="50"/>
   </link>
+    <!-- Import macro for realsense-RS200 camera-->
+    <xacro:include filename="$(find realsense_gazebo_plugin)/urdf/realsense-RS200.macro.xacro"/>
+    <!-- Create camera instance -->
+    <xacro:realsense-rs200 prefix="" parent="base_link">
+        <origin xyz=".45 0 0.2" rpy="0 0 0" />
+    </xacro:realsense-rs200>
   <xacro:macro name="m_joint" params="name type axis_xyz origin_rpy origin_xyz parent child limit_e limit_l limit_u limit_v">
     <joint name="${name}" type="${type}">
